Commit message: update code

File: mobo_bot_description/urdf/gazebo_controllers.xacro (robot description, xacro)
@@ -3,5 +3,5 @@
     <gazebo>
         <plugin name="mobo_bot_diff_drive_gazebo_control" filename="libgazebo_ros_diff_drive.so">
-            <update_rate>50</update_rate>
+            <update_rate>20</update_rate>
             <!-- wheels -->
             <left_joint>left_wheel_joint</left_joint>
@@ -11,5 +11,5 @@
             <wheel_diameter>0.1</wheel_diameter>
             <!-- limits -->
-            <max_wheel_torque>100</max_wheel_torque>
+            <max_wheel_torque>50</max_wheel_torque>
             <max_wheel_acceleration>4.0</max_wheel_acceleration>
             <command_topic>cmd_vel</command_topic>
@@ -21,5 +21,5 @@
             <odometry_frame>odom</odometry_frame>
             <!-- <odometry_source>1</odometry_source> -->
-            <robot_base_frame>base_link</robot_base_frame>
+            <robot_base_frame>base_footprint</robot_base_frame>
             <ros>
                 <!-- <namespace>/br</namespace> -->
@@ -34,5 +34,5 @@
                 <remapping>~/out:=joint_states</remapping>
             </ros>
-            <update_rate>50</update_rate>
+            <update_rate>30</update_rate>
             <joint_name>left_wheel_joint</joint_name>
             <joint_name>right_wheel_joint</joint_name>

File: mobo_bot_description/urdf/sensors/cam.xacro (robot description, xacro)
@@ -2,6 +2,6 @@
 <robot xmlns:xacro="http://www.ros.org/wiki/xacro"  name="mobo_bot">
     <!-- <xacro:arg name="cam_visual"   default="false"/> -->
-    <xacro:property name="line_sense_angle"   value="${pi/2.5}"/>
-    <xacro:property name="line_sense_mode"   value="false"/>
+    <xacro:property name="line_sense_angle"   value="${pi/2}"/>
+    <xacro:property name="line_sense_mode"   value="true"/>
     <!-- CAMERA LINK FRAME -->
     <joint name="cam_joint" type="fixed">
@@ -50,14 +50,14 @@
         <sensor type="camera" name="camera">
             <visualize>$(arg cam_visual)</visualize>
-            <update_rate>15.0</update_rate>
+            <update_rate>50.0</update_rate>
             <camera name="cam">
                 <horizontal_fov>1.4</horizontal_fov>
                 <image>
-                    <width>320</width>
-                    <height>240</height>
+                    <width>160</width>
+                    <height>120</height>
                     <format>R8G8B8</format>
                 </image>
                 <clip>
-                    <near>0.05</near>
+                    <near>0.02</near>
                     <far>5</far>
                 </clip>

File: mobo_bot_description/urdf/sensors/lidar.xacro (robot description, xacro)
@@ -4,7 +4,7 @@
     <!-- LIDAR LINK FRAME -->
     <joint name="lidar_joint" type="fixed">
-        <parent link="chassis_link"/>
+        <parent link="base_footprint"/>
         <child link="lidar_link"/>
-        <origin xyz="-0.06 0 ${chassis_height + 0.06}" rpy="0 0 0"/>
+        <origin xyz="-0.05 0 ${chassis_height + 0.11}" rpy="0 0 0"/>
         <axis xyz="0 0 0"/>
     </joint>
@@ -33,5 +33,5 @@
             <visualize>$(arg laser_visual)</visualize>
             <pose>0.0 0 0.0 0 0 0</pose>
-            <update_rate>15</update_rate>
+            <update_rate>10</update_rate>
             <ray>
                 <scan>
@@ -44,7 +44,7 @@
                 </scan>
                 <range>
-                    <min>0.15</min>
-                    <max>5</max>
-                    <resolution>0.01</resolution>
+                    <min>0.2</min>
+                    <max>4</max>
+                    <resolution>0.02</resolution>
                 </range>
                 <noise>

File: mobo_bot_description/urdf/sensors/sonar.xacro (robot description, xacro)
@@ -35,5 +35,5 @@
             <visualize>$(arg sonar_visual)</visualize>
             <pose>0.0 0 0.0 0 0 0</pose>
-            <update_rate>20</update_rate>
+            <update_rate>5</update_rate>
             <ray>
                 <scan>

File: mobo_bot_description/urdf/urdf_description.xacro (robot description, xacro)
@@ -23,17 +23,10 @@
     <!-- BASE LINK -->
     <!-- <base joint/> -->
-    <link name="base_link">
+    <link name="base_footprint">
     </link>
     <!-- ################# -->
-    <joint name="base_footprint_joint" type="fixed">
-        <parent link="base_link"/>
-        <child link="base_footprint"/>
-        <origin xyz="0 0 0" rpy="0 0 0"/>
-    </joint>
-    <link name="base_footprint">
-    </link>
     <!-- CHASSIS LINK -->
     <joint name="chassis_joint" type="fixed">
-        <parent link="base_link"/>
+        <parent link="base_footprint"/>
         <child link="chassis_link"/>
         <origin xyz="0 0 0.05"/>
@@ -57,7 +50,7 @@
     <!--  FRONT LEFT WHEEL LINK -->
     <joint name="left_wheel_joint" type="continuous">
-        <parent link="chassis_link"/>
+        <parent link="base_footprint"/>
         <child link="left_wheel_link"/>
-        <origin xyz="0 0.2 0" rpy="${-pi/2} 0 0"/>
+        <origin xyz="0 0.2 0.05" rpy="${-pi/2} 0 0"/>
         <axis xyz="0 0 1"/>
     </joint>
@@ -84,7 +77,7 @@
     <!--  FRONT RIGHT WHEEL LINK -->
     <joint name="right_wheel_joint" type="continuous">
-        <parent link="chassis_link"/>
+        <parent link="base_footprint"/>
         <child link="right_wheel_link"/>
-        <origin xyz="0 -0.2 0" rpy="${-pi/2} 0 0"/>
+        <origin xyz="0 -0.2 0.05" rpy="${-pi/2} 0 0"/>
         <axis xyz="0 0 1"/>
     </joint>
@@ -143,5 +136,5 @@
     <!--  ########################### -->
     <xacro:include filename="$(find mobo_bot_description)/urdf/gazebo_controllers.xacro"/>
-    <xacro:include filename="$(find mobo_bot_description)/urdf/sensors/imu.xacro"/>
+    <!-- <xacro:include filename="$(find mobo_bot_description)/urdf/sensors/imu.xacro"/> -->
     <xacro:include filename="$(find mobo_bot_description)/urdf/sensors/lidar.xacro"/>
     <xacro:include filename="$(find mobo_bot_description)/urdf/sensors/cam.xacro"/>
