Commit message: feat: updated sensor and core urdf

File: mobo_bot_description/urdf/robot_core.xacro (robot description, xacro)
@@ -106,5 +106,8 @@
         parent_name="chassis"
         x="${-chassis_length/4}" y="0" z="${chassis_height+lidar_z_offset}"
-        mass="0.08"/>
+        mass="0.08" samples="360"
+        min_angle="${-pi/2}" max_angle="${pi/2}"
+        min_range="0.1" max_range="10"
+        visualize="false"/>
     <!--  imu -->
     <xacro:insert_imu
@@ -117,5 +120,17 @@
         parent_name="chassis"
         x="${(chassis_length*0.375)+0.03}" y="0" z="${0.05-wheel_radius}"
-        mass="0.005" tilt_angle="${pi/2.1}"/> -->
+        mass="0.005"
+        width="320" height="240"
+        min_range="0.02" max_range="5.0"
+        tilt_angle="${pi/2.1}"
+        visualize="false"/> -->
+    <!--  front sonar sensor -->
+    <!-- <xacro:insert_sonar
+        base_name="sonar"
+        parent_name="chassis"
+        x="${(chassis_length*0.375)+0.005}" y="0" z="${(chassis_height/2)+0.04}"
+        mass="0.0005"
+        min_range="0.02" max_range="3.0"
+        resolution="0.01" visualize="false"/> -->
     <!--  normal camera style -->
     <!-- <xacro:property name="cam_x_offset" value="0.04"/>
@@ -125,10 +140,16 @@
         parent_name="chassis"
         x="${(chassis_length*0.375)+cam_x_offset}" y="0" z="${chassis_height+cam_z_offset}"
-        mass="0.005" tilt_angle="0"/> -->
+        mass="0.005"
+        width="320" height="240"
+        min_range="0.02" max_range="5.0"
+        tilt_angle="0"
+        visualize="true"/> -->
     <!--  front sonar sensor -->
     <!-- <xacro:insert_sonar
         base_name="sonar"
         parent_name="chassis"
-        x="${(chassis_length*0.375)+0.005}" y="0" z="${chassis_height/2}"
-        mass="0.0005"/> -->
+        x="${(chassis_length*0.375)+0.005}" y="0" z="${(chassis_height/2)}"
+        mass="0.0005"
+        min_range="0.02" max_range="3.0"
+        resolution="0.01" visualize="false"/> -->
 </robot>

File: mobo_bot_description/urdf/sensors/cam.xacro (robot description, xacro)
@@ -1,5 +1,5 @@
 <?xml version="1.0"?>
 <robot xmlns:xacro="http://www.ros.org/wiki/xacro" >
-    <xacro:macro name="insert_camera" params="base_name parent_name x y z mass tilt_angle">
+    <xacro:macro name="insert_camera" params="base_name parent_name x y z mass width height min_range max_range tilt_angle visualize">
         <joint name="${base_name}_joint" type="fixed">
             <parent link="${parent_name}"/>
@@ -42,16 +42,16 @@
             <material>Gazebo/DarkGrey</material>
             <sensor type="${base_name}" name="camera">
-                <visualize>false</visualize>
+                <visualize>${visualize}</visualize>
                 <update_rate>20.0</update_rate>
-                <camera name="cam">
+                <camera name="${base_name}">
                     <horizontal_fov>1.4</horizontal_fov>
                     <image>
-                        <width>320</width>
-                        <height>240</height>
+                        <width>${width}</width>
+                        <height>${height}</height>
                         <format>R8G8B8</format>
                     </image>
                     <clip>
-                        <near>0.02</near>
-                        <far>5</far>
+                        <near>${min_range}</near>
+                        <far>${max_range}</far>
                     </clip>
                     <noise>
@@ -68,5 +68,5 @@
                     </ros> -->
                     <!-- Set camera name. If empty, defaults to sensor name (i.e. "sensor_name") -->
-                    <camera_name>cam</camera_name>
+                    <camera_name>${base_name}</camera_name>
                     <!-- Set TF frame name. If empty, defaults to link name (i.e. "link_name") -->
                     <frame_name>${base_name}_optical_link</frame_name>

File: mobo_bot_description/urdf/sensors/imu.xacro (robot description, xacro)
@@ -57,5 +57,5 @@
                 <plugin name="${base_name}_plugin" filename="libgazebo_ros_imu_sensor.so">
                     <ros>
-                        <namespace>imu</namespace>
+                        <namespace>${base_name}</namespace>
                         <remapping>~/out:=data</remapping>
                     </ros>

File: mobo_bot_description/urdf/sensors/lidar.xacro (robot description, xacro)
@@ -1,5 +1,5 @@
 <?xml version="1.0"?>
 <robot xmlns:xacro="http://www.ros.org/wiki/xacro" >
-    <xacro:macro name="insert_lidar" params="base_name parent_name x y z mass">
+    <xacro:macro name="insert_lidar" params="base_name parent_name x y z mass samples min_angle max_angle min_range max_range visualize">
         <joint name="${base_name}_joint" type="fixed">
             <parent link="${parent_name}"/>
@@ -35,22 +35,24 @@
             <sensor name="${base_name}" type="ray">
                 <pose> 0 0 0 0 0 0 </pose>
-                <visualize>false</visualize>
+                <visualize>${visualize}</visualize>
                 <update_rate>10</update_rate>
                 <ray>
                     <scan>
                         <horizontal>
-                            <samples>360</samples>
-                            <min_angle>-3.14</min_angle>
-                            <max_angle>3.14</max_angle>
+                            <samples>${samples}</samples>
+                            <min_angle>${min_angle}</min_angle>
+                            <max_angle>${max_angle}</max_angle>
                         </horizontal>
                     </scan>
                     <range>
-                        <min>0.2</min>
-                        <max>10</max>
+                        <min>${min_range}</min>
+                        <max>${max_range}</max>
                     </range>
                 </ray>
-                <plugin name="${base_name}_controller" filename="libgazebo_ros_ray_sensor.so">
+                <plugin name="${base_name}_plugin" filename="libgazebo_ros_ray_sensor.so">
                     <ros>
-                        <argument>~/out:=scan</argument>
+                        <namespace>${base_name}</namespace>
+                        <remapping>~/out:=scan</remapping>
+                        <!-- <argument>~/out:=scan</argument> -->
                     </ros>
                     <output_type>sensor_msgs/LaserScan</output_type>

File: mobo_bot_description/urdf/sensors/sonar.xacro (robot description, xacro)
@@ -2,7 +2,7 @@
 <robot xmlns:xacro="http://www.ros.org/wiki/xacro">
     <!-- <xacro:arg name="sonar_visual"   default="false"/> -->
-    <xacro:property name="deg2rad" value="0.017460317"/>
-    <xacro:property name="scan_angle" value="1"/>
-    <xacro:macro name="insert_sonar" params="base_name parent_name x y z mass">
+    <!-- <xacro:property name="deg2rad" value="0.017460317"/>
+    <xacro:property name="scan_angle" value="1"/> -->
+    <xacro:macro name="insert_sonar" params="base_name parent_name x y z mass min_range max_range resolution visualize">
         <joint name="${base_name}_joint" type="fixed">
             <parent link="${parent_name}"/>
@@ -32,5 +32,5 @@
             <sensor name="${base_name}" type="ray">
                 <always_on>true</always_on>
-                <visualize>false</visualize>
+                <visualize>${visualize}</visualize>
                 <pose>0.0 0 0.0 0 0 0</pose>
                 <update_rate>5</update_rate>
@@ -38,25 +38,25 @@
                     <scan>
                         <horizontal>
-                        <samples>20</samples>
-                        <resolution>1</resolution>
-                        <min_angle>${-scan_angle * deg2rad}</min_angle>
-                        <max_angle>${scan_angle * deg2rad}</max_angle>
+                            <samples>20</samples>
+                            <resolution>1</resolution>
+                            <min_angle>${-pi/90}</min_angle>
+                            <max_angle>${pi/90}</max_angle>
                         </horizontal>
                         <vertical>
-                        <samples>20</samples>
-                        <resolution>1</resolution>
-                        <min_angle>${-scan_angle * deg2rad}</min_angle>
-                        <max_angle>${scan_angle * deg2rad}</max_angle>
+                            <samples>20</samples>
+                            <resolution>1</resolution>
+                            <min_angle>${-pi/150}</min_angle>
+                            <max_angle>${pi/150}</max_angle>
                         </vertical>
                     </scan>
                     <range>
-                        <min>0.01</min>
-                        <max>2</max>
-                        <resolution>0.02</resolution>
+                        <min>${min_range}</min>
+                        <max>${max_range}</max>
+                        <resolution>${resolution}</resolution>
                     </range>
                 </ray>
                 <plugin name="${base_name}_plugin" filename="libgazebo_ros_ray_sensor.so">
                     <ros>
-                        <namespace>sonar</namespace>
+                        <namespace>${base_name}</namespace>
                         <remapping>~/out:=range</remapping>
                     </ros>
