Commit message: fix: solved wheel rim display problem

File: mobo_bot_description/urdf/color_macros.xacro (robot description, xacro)
@@ -1,4 +1,4 @@
 <?xml version="1.0"?>
-<robot name="mobo_bot" xmlns:xacro="http://www.ros.org/wiki/xacro" >
+<robot xmlns:xacro="http://www.ros.org/wiki/xacro" >
     <material name="white">
         <color rgba="1 1 1 1" />

File: mobo_bot_description/urdf/controllers/gazebo_control.xacro (robot description, xacro)
@@ -1,4 +1,4 @@
 <?xml version="1.0"?>
-<robot name="mobo_bot" xmlns:xacro="http://ros.org/wiki/xacro">
+<robot xmlns:xacro="http://ros.org/wiki/xacro">
     <gazebo>
         <plugin name="mobo_bot_diff_drive_gazebo_control" filename="libgazebo_ros_diff_drive.so">

File: mobo_bot_description/urdf/controllers/gazebo_hw_ros2_control.xacro (robot description, xacro)
@@ -1,4 +1,4 @@
 <?xml version="1.0"?>
-<robot name="mobo_bot" xmlns:xacro="http://www.ros.org/wiki/xacro">
+<robot xmlns:xacro="http://www.ros.org/wiki/xacro">
     <xacro:include filename="transmission_macros.xacro"/>
     <ros2_control name="mobo_bot_diff_drive_gazebo_hw_ros2_control" type="system">

File: mobo_bot_description/urdf/inertia_macros.xacro (robot description, xacro)
@@ -1,4 +1,4 @@
 <?xml version="1.0"?>
-<robot name="mobo_bot" xmlns:xacro="http://www.ros.org/wiki/xacro" >
+<robot xmlns:xacro="http://www.ros.org/wiki/xacro" >
     <!-- Specify some standard inertial calculations https://en.wikipedia.org/wiki/List_of_moments_of_inertia -->
     <!-- These make use of xacro's mathematical functionality -->

File: mobo_bot_description/urdf/other_parts/box_with_fillet_macro.xacro (robot description, xacro)
@@ -1,4 +1,4 @@
 <?xml version="1.0"?>
-<robot name="mobo_bot" xmlns:xacro="http://www.ros.org/wiki/xacro" >
+<robot xmlns:xacro="http://www.ros.org/wiki/xacro" >
     <xacro:macro name="insert_box_with_fillet" params="x y z size_x size_y size_z fillet_radius material">
             <!-- logitudinal box -->

File: mobo_bot_description/urdf/other_parts/drive_wheel_macro.xacro (robot description, xacro)
@@ -1,12 +1,7 @@
 <?xml version="1.0"?>
-<robot name="mobo_bot" xmlns:xacro="http://www.ros.org/wiki/xacro" >
+<robot xmlns:xacro="http://www.ros.org/wiki/xacro" >
     <xacro:macro name="material_black">
         <material name="black">
             <color rgba="0.1 0.1 0.1 1"/>
-        </material>
-    </xacro:macro>
-    <xacro:macro name="material_red">
-        <material name="red">
-            <color rgba="1 0 0 1"/>
         </material>
     </xacro:macro>
@@ -33,5 +28,5 @@
     </xacro:macro>
     <!--  ########################### -->
-    <xacro:macro name="insert_drive_wheel" params="base_name parent_name x y z mass radius thickness spoke_width">
+    <xacro:macro name="insert_drive_wheel" params="base_name parent_name x y z mass radius thickness">
         <joint name="${base_name}_joint" type="continuous">
             <parent link="${parent_name}"/>
@@ -60,42 +55,4 @@
         </link>
         <xacro:gazebo_wheel_settings name="${base_name}"/>
-        <joint name="${base_name}_rim_joint" type="fixed">
-            <parent link="${base_name}"/>
-            <child link="${base_name}_rim"/>
-            <origin xyz="0 0 0" rpy="0 0 0"/>
-        </joint>
-        <link name="${base_name}_rim">
-            <visual>
-                <origin xyz="0 0 0" rpy="0 0 0"/>
-                <geometry>
-                    <box size="${spoke_width} ${radius*1.2} ${thickness+0.005}"/>
-                </geometry>
-                <xacro:material_red/>
-            </visual>
-            <visual>
-                <origin xyz="0 0 0" rpy="0 0 ${pi/2}"/>
-                <geometry>
-                    <box size="${spoke_width} ${radius*1.2} ${thickness+0.005}"/>
-                </geometry>
-                <xacro:material_red/>
-            </visual>
-            <visual>
-                <origin xyz="0 0 0" rpy="0 0 ${-pi/4}"/>
-                <geometry>
-                    <box size="${spoke_width} ${radius*1.2} ${thickness+0.005}"/>
-                </geometry>
-                <xacro:material_red/>
-            </visual>
-            <visual>
-                <origin xyz="0 0 0" rpy="0 0 ${pi/4}"/>
-                <geometry>
-                    <box size="${spoke_width} ${radius*1.2} ${thickness+0.005}"/>
-                </geometry>
-                <xacro:material_red/>
-            </visual>
-        </link>
-        <gazebo reference="${base_name}_rim">
-            <material>Gazebo/Red</material>
-        </gazebo>
     </xacro:macro>
 </robot>

File: mobo_bot_description/urdf/robot_core.xacro (robot description, xacro)
@@ -1,6 +1,7 @@
 <?xml version="1.0"?>
-<robot name="mobo_bot" xmlns:xacro="http://www.ros.org/wiki/xacro">
+<robot xmlns:xacro="http://www.ros.org/wiki/xacro">
     <xacro:include filename="other_parts/box_with_fillet_macro.xacro"/>
     <xacro:include filename="other_parts/drive_wheel_macro.xacro"/>
+    <xacro:include filename="other_parts/drive_wheel_rim_macro.xacro"/>
     <xacro:include filename="sensors/sonar.xacro"/>
     <xacro:include filename="sensors/lidar.xacro"/>
@@ -8,6 +9,6 @@
     <!-- <xacro:include filename="sensors/cam.xacro"/> -->
     <xacro:property name="chassis_length" value="0.25"/>
-    <xacro:property name="chassis_width" value="0.18"/>
-    <xacro:property name="chassis_height" value="0.09"/>
+    <xacro:property name="chassis_width" value="0.19"/>
+    <xacro:property name="chassis_height" value="0.07"/>
     <xacro:property name="chassis_mass" value="3.0"/>
     <xacro:property name="wheel_seperation" value="0.214"/>
@@ -26,10 +27,10 @@
         <parent link="base_link"/>
         <child link="chassis"/>
-        <origin xyz="0 0 ${wheel_radius*2}"/>
+        <origin xyz="0 0 ${(wheel_radius*2)+0.002}"/>
     </joint>
     <link name="chassis">
         <xacro:insert_box_with_fillet x="${-chassis_length/6}" y="0" z="${chassis_height/2}"
             size_x="${chassis_length}" size_y="${chassis_width}" size_z="${chassis_height}"
-            fillet_radius="0.04" material="orange"/>
+            fillet_radius="0.05" material="orange"/>
         <collision>
            <origin xyz="${-chassis_length/6} 0 ${chassis_height/2}" rpy="0 0 0"/>
@@ -45,29 +46,42 @@
         <material>Gazebo/Orange</material>
     </gazebo>
-    <!-- <xacro:insert_face parent_name="chassis" x="${(chassis_length/6)*2}" y="0" z="${chassis_height/2}"/> -->
     <!--  ########################### -->
-    <!-- LEFT AND RIGHT DRIVE WHEELS -->
+    <!-- LEFT DRIVE WHEEL -->
     <xacro:insert_drive_wheel
         base_name="left_wheel"
-        parent_name="chassis"
-        x="0" y="${wheel_seperation/2}" z="${-wheel_radius}"
+        parent_name="base_link"
+        x="0" y="${wheel_seperation/2}" z="${wheel_radius}"
         mass="${wheel_mass}"
+        radius="${wheel_radius}"
+        thickness="${wheel_width}"/>
+    <xacro:insert_drive_wheel_rim
+        base_name="left_rim"
+        parent_name="left_wheel"
+        x="0" y="0" z="0.001"
         radius="${wheel_radius}"
         thickness="${wheel_width}"
         spoke_width="0.005"/>
+    <!-- ############################# -->
+    <!-- RIGHT DRIVE WHEEL -->
     <xacro:insert_drive_wheel
         base_name="right_wheel"
-        parent_name="chassis"
-        x="0" y="${-wheel_seperation/2}" z="${-wheel_radius}"
+        parent_name="base_link"
+        x="0" y="${-wheel_seperation/2}" z="${wheel_radius}"
         mass="${wheel_mass}"
+        radius="${wheel_radius}"
+        thickness="${wheel_width}"/>
+    <xacro:insert_drive_wheel_rim
+        base_name="right_rim"
+        parent_name="right_wheel"
+        x="0" y="0" z="-0.001"
         radius="${wheel_radius}"
         thickness="${wheel_width}"
         spoke_width="0.005"/>
-    <!-- ############################### -->
+    <!-- ############################# -->
     <!--  castor WHEEL LINK -->
     <joint name="castor_wheel_joint" type="fixed">
-        <parent link="chassis"/>
+        <parent link="base_link"/>
         <child link="castor_wheel"/>
-        <origin xyz="${-chassis_length/2} 0 ${-1*((wheel_radius*2)-castor_wheel_radius)}"/>
+        <origin xyz="${-chassis_length/2} 0 ${castor_wheel_radius}"/>
     </joint>
     <link name="castor_wheel">
@@ -104,5 +118,5 @@
         parent_name="chassis"
         x="${(chassis_length/6)*2}" y="0" z="${chassis_height/2}"
-        mass="0.0005"
+        mass="0.005"
         min_range="0.02" max_range="3.0"
         resolution="0.01" visualize="false"/>
