Commit message: feat: update sensor and part xaro files

File: mobo_bot_description/urdf/other_parts/box_with_fillet_macro.xacro (robot description, xacro)
@@ -1,5 +1,5 @@
 <?xml version="1.0"?>
 <robot name="mobo_bot" xmlns:xacro="http://www.ros.org/wiki/xacro" >
-    <xacro:macro name="box_with_fillet" params="x y z size_x size_y size_z fillet_radius material">
+    <xacro:macro name="insert_box_with_fillet" params="x y z size_x size_y size_z fillet_radius material">
             <!-- logitudinal box -->
             <visual>

File: mobo_bot_description/urdf/other_parts/face_macro.xacro (robot description, xacro)
@@ -1,34 +1,37 @@
 <?xml version="1.0"?>
 <robot name="mobo_bot" xmlns:xacro="http://www.ros.org/wiki/xacro" >
-    <joint name="face_joint" type="fixed">
-        <parent link="chassis"/>
-        <child link="face_link"/>
-        <origin xyz="${chassis_length} 0 ${chassis_height/2}" rpy="0 0 0"/>
-    </joint>
-    <link name="face_link">
-        <visual>
-            <origin xyz="0 0.05 0.01" rpy="0 ${pi/2} 0"/>
-            <geometry>
-                <cylinder radius="0.01" length="0.002"/>
-            </geometry>
-            <material name="black"/>
-        </visual>
-        <visual>
-            <origin xyz="0 -0.05 0.01" rpy="0 ${pi/2} 0"/>
-            <geometry>
-                <cylinder radius="0.01" length="0.002"/>
-            </geometry>
-            <material name="black"/>
-        </visual>
-        <visual>
-            <origin xyz="-0.011 0 -0.00" rpy="0 ${1.5} 0"/>
-            <geometry>
-                <cylinder radius="0.05" length="0.02"/>
-            </geometry>
-            <material name="black"/>
-        </visual>
-    </link>
-    <gazebo reference="face_link">
-        <material>Gazebo/FlatBlack</material>
-    </gazebo>
+    <xacro:macro name="insert_face" params="parent_name x y z">
+        <joint name="face_joint" type="fixed">
+            <parent link="${parent_name}"/>
+            <child link="face_link"/>
+            <origin xyz="${x} ${y} ${z}" rpy="0 0 0"/>
+            <!-- <origin xyz="${chassis_length} 0 ${chassis_height/2}" rpy="0 0 0"/> -->
+        </joint>
+        <link name="face_link">
+            <visual>
+                <origin xyz="0 0.05 0.01" rpy="0 ${pi/2} 0"/>
+                <geometry>
+                    <cylinder radius="0.01" length="0.002"/>
+                </geometry>
+                <material name="black"/>
+            </visual>
+            <visual>
+                <origin xyz="0 -0.05 0.01" rpy="0 ${pi/2} 0"/>
+                <geometry>
+                    <cylinder radius="0.01" length="0.002"/>
+                </geometry>
+                <material name="black"/>
+            </visual>
+            <visual>
+                <origin xyz="-0.011 0 -0.00" rpy="0 ${1.5} 0"/>
+                <geometry>
+                    <cylinder radius="0.05" length="0.02"/>
+                </geometry>
+                <material name="black"/>
+            </visual>
+        </link>
+        <gazebo reference="face_link">
+            <material>Gazebo/FlatBlack</material>
+        </gazebo>
+    </xacro:macro>
 </robot>

File: mobo_bot_description/urdf/robot_core.xacro (robot description, xacro)
@@ -1,7 +1,11 @@
 <?xml version="1.0"?>
 <robot name="mobo_bot" xmlns:xacro="http://www.ros.org/wiki/xacro">
-    <xacro:include filename="other_parts/fillet_box_macro.xacro"/>
-    <xacro:include filename="other_parts/insert_drive_wheel_macro.xacro"/>
-    <xacro:include filename="other_parts/insert_castor_wheel_macro.xacro"/>
+    <xacro:include filename="other_parts/box_with_fillet_macro.xacro"/>
+    <xacro:include filename="other_parts/drive_wheel_macro.xacro"/>
+    <xacro:include filename="other_parts/face_macro.xacro"/>
+    <xacro:include filename="sensors/lidar.xacro"/>
+    <xacro:include filename="sensors/imu.xacro"/>
+    <xacro:include filename="sensors/cam.xacro"/>
+    <xacro:include filename="sensors/sonar.xacro"/>
     <xacro:property name="chassis_height" value="0.125"/>
     <xacro:property name="chassis_length" value="0.3"/>
@@ -26,5 +30,7 @@
     </joint>
     <link name="chassis">
-        <xacro:box_with_fillet x="${-chassis_length/8}" y="0" z="${chassis_height/2}" size_x="${chassis_length}" size_y="${chassis_width}" size_z="${chassis_height}" fillet_radius="0.05" material="orange"/>
+        <xacro:insert_box_with_fillet x="${-chassis_length/8}" y="0" z="${chassis_height/2}"
+            size_x="${chassis_length}" size_y="${chassis_width}" size_z="${chassis_height}"
+            fillet_radius="0.05" material="orange"/>
         <collision>
            <origin xyz="${-chassis_length/8} 0 ${chassis_height/2}" rpy="0 0 0"/>
@@ -40,5 +46,7 @@
         <material>Gazebo/Orange</material>
     </gazebo>
+    <xacro:insert_face parent_name="chassis" x="${(chassis_length/8)*3}" y="0" z="${chassis_height/2}"/>
     <!--  ########################### -->
+    <!-- LEFT AND RIGHT DRIVE WHEELS -->
     <xacro:insert_drive_wheel
         base_name="left_wheel"
@@ -57,4 +65,5 @@
         thickness="${wheel_width}"
         spoke_width="0.005"/>
+    <!-- ############################### -->
     <!--  castor WHEEL LINK -->
     <joint name="castor_wheel_joint" type="fixed">
@@ -69,5 +78,5 @@
                 <sphere radius="${wheel_radius/2}" />
             </geometry>
-            <material name="grey"/>
+            <material name="silver"/>
         </visual>
         <collision>
@@ -88,6 +97,38 @@
         <!-- <fdir1>1 0 0</fdir1> -->
         <!-- <minDepth>0.01</minDepth> -->
-        <material>Gazebo/Grey</material>
+        <material>Gazebo/Silver</material>
     </gazebo>
     <!--  ########################### -->
+    <!--  lidar -->
+    <xacro:property name="lidar_z_offset" value="0.1"/>
+    <xacro:insert_lidar
+        base_name="lidar"
+        parent_name="chassis"
+        x="${-chassis_length/4}" y="0" z="${chassis_height+lidar_z_offset}"
+        mass="0.08"/>
+    <!--  imu -->
+    <xacro:insert_imu
+        base_name="imu"
+        parent_name="chassis"
+        x="0" y="0" z="${chassis_height}"/>
+    <!--  line tracking camera style -->
+    <!-- <xacro:insert_camera
+        base_name="line_cam"
+        parent_name="chassis"
+        x="${(chassis_length*0.375)+0.03}" y="0" z="${0.05-wheel_radius}"
+        mass="0.005" tilt_angle="${pi/2.1}"/> -->
+    <!--  normal camera style -->
+    <!-- <xacro:property name="cam_x_offset" value="0.04"/>
+    <xacro:property name="cam_z_offset" value="0.02"/>
+    <xacro:insert_camera
+        base_name="line_cam"
+        parent_name="chassis"
+        x="${(chassis_length*0.375)+cam_x_offset}" y="0" z="${chassis_height+cam_z_offset}"
+        mass="0.005" tilt_angle="0"/> -->
+    <!--  front sonar sensor -->
+    <!-- <xacro:insert_sonar
+        base_name="sonar"
+        parent_name="chassis"
+        x="${(chassis_length*0.375)+0.005}" y="0" z="${chassis_height/2}"
+        mass="0.0005"/> -->
 </robot>

File: mobo_bot_description/urdf/robot_urdf.xacro (robot description, xacro)
@@ -3,5 +3,5 @@
     <!-- ########### ARGUMENTS ######################### -->
     <xacro:arg name="use_ros2_control" default="false"/>
-    <xacro:arg name="gazebo_visual" default="true"/>
+    <!-- <xacro:arg name="gazebo_visual" default="true"/> -->
     <!-- <xacro:arg name="laser_visual" default="false"/> -->
     <!-- <xacro:arg name="imu_visual"   default="true"/> -->

File: mobo_bot_description/urdf/sensors/cam.xacro (robot description, xacro)
@@ -1,84 +1,78 @@
 <?xml version="1.0"?>
-<robot xmlns:xacro="http://www.ros.org/wiki/xacro"  name="mobo_bot">
-    <!-- <xacro:arg name="cam_visual"   default="false"/> -->
-    <xacro:property name="line_sense_angle"   value="${pi/2}"/>
-    <xacro:property name="line_sense_mode"   value="true"/>
-    <!-- CAMERA LINK FRAME -->
-    <joint name="cam_joint" type="fixed">
-        <parent link="chassis_link"/>
-        <child link="cam_link"/>
-        <xacro:if value="${line_sense_mode}">
-            <origin xyz="0.16 0 0" rpy="0 ${line_sense_angle} 0"/>
-        </xacro:if>
-        <xacro:unless value="${line_sense_mode}">
-            <origin xyz="0.16 0 ${chassis_height+0.01}" rpy="0 ${pi/4} 0"/>
-        </xacro:unless>
-    </joint>
-    <link name="cam_link">
-        <visual>
-            <origin xyz="-0.005 0 0" rpy="0 ${pi/2} 0"/>
-            <geometry>
-                <cylinder radius="0.01" length="0.01"/>
-            </geometry>
-            <material name="grey"/>
-        </visual>
-        <visual>
-            <origin xyz="-0.015 0 0" rpy="0 0 0"/>
-            <geometry>
-                <box size="0.01 0.04 0.025" />
-            </geometry>
-            <material name="grey"/>
-        </visual>
-        <collision>
-            <origin xyz="-0.01 0 0" rpy="0 0 0"/>
-            <geometry>
-                <box size="0.02 0.04 0.025"/>
-            </geometry>
-        </collision>
-        <xacro:inertial_box mass="0.0005" x="0.02" y="0.04" z="0.025">
-            <origin xyz="-0.01 0 0" rpy="0 0 0"/>
-        </xacro:inertial_box>
-    </link>
-    <joint name="cam_optical_joint" type="fixed">
-        <parent link="cam_link"/>
-        <child link="cam_optical_link"/>
-        <origin xyz="0 0 0" rpy="${-pi/2} 0 ${-pi/2}"/>
-    </joint>
-    <link name="cam_optical_link"/>
-    <gazebo reference="cam_link">
-        <material>Gazebo/DarkGrey</material>
-        <sensor type="camera" name="camera">
-            <visualize>$(arg cam_visual)</visualize>
-            <update_rate>50.0</update_rate>
-            <camera name="cam">
-                <horizontal_fov>1.4</horizontal_fov>
-                <image>
-                    <width>160</width>
-                    <height>120</height>
-                    <format>R8G8B8</format>
-                </image>
-                <clip>
-                    <near>0.02</near>
-                    <far>5</far>
-                </clip>
-                <noise>
-                    <type>gaussian</type>
-                    <mean>0.0</mean>
-                    <stddev>0.007</stddev>
-                </noise>
-            </camera>
-            <plugin name="rgb_cam_plugin" filename="libgazebo_ros_camera.so">
-                <!-- <ros>
-                    <namespace>cam</namespace>
-                    <remapping>~/image_raw:=raw</remapping>
-                    <remapping>~/camera_info:=info</remapping>
-                </ros> -->
-                <!-- Set camera name. If empty, defaults to sensor name (i.e. "sensor_name") -->
-                <camera_name>cam</camera_name>
-                <!-- Set TF frame name. If empty, defaults to link name (i.e. "link_name") -->
-                <frame_name>cam_optical_link</frame_name>
-                <hack_baseline>0.2</hack_baseline>
-            </plugin>
-        </sensor>
-    </gazebo>
+<robot xmlns:xacro="http://www.ros.org/wiki/xacro" >
+    <xacro:macro name="insert_camera" params="base_name parent_name x y z mass tilt_angle">
+        <joint name="${base_name}_joint" type="fixed">
+            <parent link="${parent_name}"/>
+            <child link="${base_name}"/>
+            <origin xyz="${x} ${y} ${z}" rpy="0 ${tilt_angle} 0"/>
+        </joint>
+        <link name="${base_name}">
+            <visual>
+                <origin xyz="-0.02 0 0" rpy="0 ${-pi/2} 0"/>
+                <geometry>
+                    <cylinder radius="0.015" length="0.04"/>
+                </geometry>
+                <material name="grey"/>
+            </visual>
+            <visual>
+                <origin xyz="-0.03 0 0" rpy="0 ${-pi/2} 0"/>
+                <geometry>
+                    <!-- <cylinder radius="0.03" length="0.02"/> -->
+                    <box size="0.04 0.06 0.02"/>
+                </geometry>
+                <material name="grey"/>
+            </visual>
+            <collision>
+                <origin xyz="-0.02 0 0" rpy="0 ${-pi/2} 0"/>
+                <geometry>
+                    <cylinder radius="0.02" length="0.04"/>
+                </geometry>
+            </collision>
+            <xacro:inertial_cylinder mass="${mass}" radius="0.02" length="0.04">
+                <origin xyz="-0.02 0 0" rpy="0 ${-pi/2} 0"/>
+            </xacro:inertial_cylinder>
+        </link>
+        <joint name="${base_name}_optical_joint" type="fixed">
+            <parent link="${base_name}"/>
+            <child link="${base_name}_optical_link"/>
+            <origin xyz="0 0 0" rpy="${-pi/2} 0 ${-pi/2}"/>
+        </joint>
+        <link name="${base_name}_optical_link"/>
+        <gazebo reference="${base_name}">
+            <material>Gazebo/DarkGrey</material>
+            <sensor type="${base_name}" name="camera">
+                <visualize>false</visualize>
+                <update_rate>20.0</update_rate>
+                <camera name="cam">
+                    <horizontal_fov>1.4</horizontal_fov>
+                    <image>
+                        <width>320</width>
+                        <height>240</height>
+                        <format>R8G8B8</format>
+                    </image>
+                    <clip>
+                        <near>0.02</near>
+                        <far>5</far>
+                    </clip>
+                    <noise>
+                        <type>gaussian</type>
+                        <mean>0.0</mean>
+                        <stddev>0.007</stddev>
+                    </noise>
+                </camera>
+                <plugin name="${base_name}_plugin" filename="libgazebo_ros_camera.so">
+                    <!-- <ros>
+                        <namespace>cam</namespace>
+                        <remapping>~/image_raw:=raw</remapping>
+                        <remapping>~/camera_info:=info</remapping>
+                    </ros> -->
+                    <!-- Set camera name. If empty, defaults to sensor name (i.e. "sensor_name") -->
+                    <camera_name>cam</camera_name>
+                    <!-- Set TF frame name. If empty, defaults to link name (i.e. "link_name") -->
+                    <frame_name>${base_name}_optical_link</frame_name>
+                    <hack_baseline>0.2</hack_baseline>
+                </plugin>
+            </sensor>
+        </gazebo>
+    </xacro:macro>
 </robot>

File: mobo_bot_description/urdf/sensors/imu.xacro (robot description, xacro)
@@ -1,69 +1,68 @@
 <?xml version="1.0"?>
-<robot xmlns:xacro="http://www.ros.org/wiki/xacro"  name="mobo_bot">
-    <!-- <xacro:arg name="imu_visual"   default="true"/> -->
-  <!-- IMU LINK FRAME -->
-    <joint name="imu_joint" type="fixed">
-        <parent link="chassis_link"/>
-        <child link="imu_link"/>
-        <origin xyz="0 0 ${chassis_height}" rpy="0 0 0"/>
-        <axis xyz="0 0 0"/>
-    </joint>
-    <link name="imu_link"/>
-    <gazebo reference="imu_link">
-        <sensor name="imu" type="imu">
-            <always_on>true</always_on>
-            <update_rate>30</update_rate>
-            <visualize>$(arg imu_visual)</visualize>
-            <imu>
-            <angular_velocity>
-                <x>
-                <noise type="gaussian">
-                    <mean>0.0</mean>
-                    <stddev>2e-4</stddev>
-                </noise>
-                </x>
-                <y>
-                <noise type="gaussian">
-                    <mean>0.0</mean>
-                    <stddev>2e-4</stddev>
-                </noise>
-                </y>
-                <z>
-                <noise type="gaussian">
-                    <mean>0.0</mean>
-                    <stddev>2e-4</stddev>
-                </noise>
-                </z>
-            </angular_velocity>
-            <linear_acceleration>
-                <x>
-                <noise type="gaussian">
-                    <mean>0.0</mean>
-                    <stddev>1.7e-2</stddev>
-                </noise>
-                </x>
-                <y>
-                <noise type="gaussian">
-                    <mean>0.0</mean>
-                    <stddev>1.7e-2</stddev>
-                </noise>
-                </y>
-                <z>
-                <noise type="gaussian">
-                    <mean>0.0</mean>
-                    <stddev>1.7e-2</stddev>
-                </noise>
-                </z>
-            </linear_acceleration>
-            </imu>
-            <plugin name="imu_plugin" filename="libgazebo_ros_imu_sensor.so">
-                <ros>
-                    <namespace>imu</namespace>
-                    <remapping>~/out:=data</remapping>
-                </ros>
-                <initial_orientation_as_reference>false</initial_orientation_as_reference>
-                <frame_name>imu_link</frame_name>
-            </plugin>
-        </sensor>
-    </gazebo>
+<robot xmlns:xacro="http://www.ros.org/wiki/xacro">
+    <xacro:macro name="insert_imu" params="base_name parent_name x y z">
+        <joint name="${base_name}_joint" type="fixed">
+            <parent link="${parent_name}"/>
+            <child link="${base_name}"/>
+            <origin xyz="${x} ${y} ${z}" rpy="0 0 0"/>
+        </joint>
+        <link name="${base_name}"/>
+        <gazebo reference="${base_name}">
+            <sensor name="${base_name}" type="imu">
+                <always_on>true</always_on>
+                <update_rate>30</update_rate>
+                <visualize>true</visualize>
+                <imu>
+                    <angular_velocity>
+                        <x>
+                            <noise type="gaussian">
+                                <mean>0.0</mean>
+                                <stddev>2e-4</stddev>
+                            </noise>
+                        </x>
+                        <y>
+                            <noise type="gaussian">
+                                <mean>0.0</mean>
+                                <stddev>2e-4</stddev>
+                            </noise>
+                        </y>
+                        <z>
+                            <noise type="gaussian">
+                                <mean>0.0</mean>
+                                <stddev>2e-4</stddev>
+                            </noise>
+                        </z>
+                    </angular_velocity>
+                    <linear_acceleration>
+                        <x>
+                            <noise type="gaussian">
+                                <mean>0.0</mean>
+                                <stddev>1.7e-2</stddev>
+                            </noise>
+                        </x>
+                        <y>
+                            <noise type="gaussian">
+                                <mean>0.0</mean>
+                                <stddev>1.7e-2</stddev>
+                            </noise>
+                        </y>
+                        <z>
+                            <noise type="gaussian">
+                                <mean>0.0</mean>
+                                <stddev>1.7e-2</stddev>
+                            </noise>
+                        </z>
+                    </linear_acceleration>
+                </imu>
+                <plugin name="${base_name}_plugin" filename="libgazebo_ros_imu_sensor.so">
+                    <ros>
+                        <namespace>imu</namespace>
+                        <remapping>~/out:=data</remapping>
+                    </ros>
+                    <initial_orientation_as_reference>false</initial_orientation_as_reference>
+                    <frame_name>${base_name}</frame_name>
+                </plugin>
+            </sensor>
+        </gazebo>
+    </xacro:macro>
 </robot>
