Commit message: feat: update sensor and part xaro files

File: mobo_bot_description/urdf/sensors/lidar.xacro (robot description, xacro)
@@ -1,66 +1,62 @@
 <?xml version="1.0"?>
-<robot xmlns:xacro="http://www.ros.org/wiki/xacro"  name="mobo_bot">
-    <!-- <xacro:arg name="laser_visual" default="false"/> -->
-    <!-- LIDAR LINK FRAME -->
-    <joint name="lidar_joint" type="fixed">
-        <parent link="base_footprint"/>
-        <child link="lidar_link"/>
-        <origin xyz="-0.05 0 ${chassis_height + 0.11}" rpy="0 0 0"/>
-        <axis xyz="0 0 0"/>
-    </joint>
-    <link name="lidar_link">
-    <visual>
-      <origin xyz="0 0 -0.02" rpy="0 0 0"/>
-      <geometry>
-        <cylinder radius="0.05" length="0.07" />
-      </geometry>
-      <material name="grey"/>
-    </visual>
-    <collision>
-      <origin xyz="0 0 -0.02" rpy="0 0 0"/>
-      <geometry>
-        <cylinder radius="0.05" length="0.07" />
-      </geometry>
-    </collision>
-    <xacro:inertial_cylinder mass="0.2" length="0.07" radius="0.05">
-            <origin xyz="0 0 -0.02" rpy="0 0 0"/>
-        </xacro:inertial_cylinder>
-    </link>
-    <gazebo reference="lidar_link">
-        <material>Gazebo/DarkGrey</material>
-        <sensor name="lidar" type="ray">
-            <always_on>true</always_on>
-            <visualize>$(arg laser_visual)</visualize>
-            <pose>0.0 0 0.0 0 0 0</pose>
-            <update_rate>10</update_rate>
-            <ray>
-                <scan>
-                <horizontal>
-                    <samples>360</samples>
-                    <resolution>1</resolution>
-                    <min_angle>${0*pi}</min_angle>
-                    <max_angle>${2*pi}</max_angle>
-                </horizontal>
-                </scan>
-                <range>
-                    <min>0.2</min>
-                    <max>4</max>
-                    <resolution>0.02</resolution>
-                </range>
-                <noise>
-                    <type>gaussian</type>
-                    <mean>0.0</mean>
-                    <stddev>0.01</stddev>
-                </noise>
-            </ray>
-            <plugin name="laser_plugin" filename="libgazebo_ros_ray_sensor.so">
-            <ros>
-                <!-- <namespace>lidar</namespace> -->
-                <remapping>~/out:=scan</remapping>
-            </ros>
-            <output_type>sensor_msgs/LaserScan</output_type>
-            <frame_name>lidar_link</frame_name>
-            </plugin>
-        </sensor>
-    </gazebo>
+<robot xmlns:xacro="http://www.ros.org/wiki/xacro" >
+    <xacro:macro name="insert_lidar" params="base_name parent_name x y z mass">
+        <joint name="${base_name}_joint" type="fixed">
+            <parent link="${parent_name}"/>
+            <child link="${base_name}"/>
+            <origin xyz="${x} ${y} ${z}" rpy="0 0 0"/>
+        </joint>
+        <link name="${base_name}">
+            <visual>
+                <origin xyz="0 0 0"/>
+                <geometry>
+                    <cylinder radius="0.05" length="0.04"/>
+                </geometry>
+                <material name="black"/>
+            </visual>
+            <visual>
+                <origin xyz="0 0 -0.05"/>
+                <geometry>
+                    <cylinder radius="0.01" length="0.1"/>
+                </geometry>
+                <material name="black"/>
+            </visual>
+            <collision>
+                <geometry>
+                    <cylinder radius="0.05" length="0.04"/>
+                </geometry>
+            </collision>
+            <xacro:inertial_cylinder mass="${mass}" length="0.04" radius="0.05">
+                <origin xyz="0 0 0" rpy="0 0 0"/>
+            </xacro:inertial_cylinder>
+        </link>
+        <gazebo reference="${base_name}">
+            <material>Gazebo/DarkGrey</material>
+            <sensor name="${base_name}" type="ray">
+                <pose> 0 0 0 0 0 0 </pose>
+                <visualize>false</visualize>
+                <update_rate>10</update_rate>
+                <ray>
+                    <scan>
+                        <horizontal>
+                            <samples>360</samples>
+                            <min_angle>-3.14</min_angle>
+                            <max_angle>3.14</max_angle>
+                        </horizontal>
+                    </scan>
+                    <range>
+                        <min>0.2</min>
+                        <max>10</max>
+                    </range>
+                </ray>
+                <plugin name="${base_name}_controller" filename="libgazebo_ros_ray_sensor.so">
+                    <ros>
+                        <argument>~/out:=scan</argument>
+                    </ros>
+                    <output_type>sensor_msgs/LaserScan</output_type>
+                    <frame_name>${base_name}</frame_name>
+                </plugin>
+            </sensor>
+        </gazebo>
+    </xacro:macro>
 </robot>

File: mobo_bot_description/urdf/sensors/sonar.xacro (robot description, xacro)
@@ -1,70 +1,70 @@
 <?xml version="1.0"?>
-<robot xmlns:xacro="http://www.ros.org/wiki/xacro"  name="mobo_bot">
+<robot xmlns:xacro="http://www.ros.org/wiki/xacro">
     <!-- <xacro:arg name="sonar_visual"   default="false"/> -->
     <xacro:property name="deg2rad" value="0.017460317"/>
     <xacro:property name="scan_angle" value="1"/>
-  <!-- SONAR LINK FRAME -->
-    <joint name="sonar_joint" type="fixed">
-        <parent link="chassis_link"/>
-        <child link="sonar_link"/>
-        <origin xyz="0.16 0 ${chassis_height/2}" rpy="0 0 0"/>
-        <axis xyz="0 0 0"/>
-    </joint>
-    <link name="sonar_link">
-        <visual>
-            <origin xyz="-0.005 0 0" rpy="0 ${pi/2} 0"/>
-            <geometry>
-                <cylinder radius="0.015" length="0.01" />
-            </geometry>
-            <material name="blue"/>
-        </visual>
-        <collision>
-            <origin xyz="-0.005 0 0" rpy="0 ${pi/2} 0"/>
-            <geometry>
-                <cylinder radius="0.015" length="0.01" />
-            </geometry>
-        </collision>
-        <xacro:inertial_cylinder mass="0.0005" length="0.01" radius="0.01">
-            <origin xyz="-0.005 0 0" rpy="0 0 0"/>
-        </xacro:inertial_cylinder>
-    </link>
-    <gazebo reference="sonar_link">
-        <material>Gazebo/Blue</material>
-        <sensor name="sonar" type="ray">
-            <always_on>true</always_on>
-            <visualize>$(arg sonar_visual)</visualize>
-            <pose>0.0 0 0.0 0 0 0</pose>
-            <update_rate>5</update_rate>
-            <ray>
-                <scan>
-                    <horizontal>
-                    <samples>20</samples>
-                    <resolution>1</resolution>
-                    <min_angle>${-scan_angle * deg2rad}</min_angle>
-                    <max_angle>${scan_angle * deg2rad}</max_angle>
-                    </horizontal>
-                    <vertical>
-                    <samples>20</samples>
-                    <resolution>1</resolution>
-                    <min_angle>${-scan_angle * deg2rad}</min_angle>
-                    <max_angle>${scan_angle * deg2rad}</max_angle>
-                    </vertical>
-                </scan>
-                <range>
-                    <min>0.01</min>
-                    <max>2</max>
-                    <resolution>0.02</resolution>
-                </range>
-            </ray>
-            <plugin name="sonar_plugin" filename="libgazebo_ros_ray_sensor.so">
-                <ros>
-                    <namespace>sonar</namespace>
-                    <remapping>~/out:=range</remapping>
-                </ros>
-                <output_type>sensor_msgs/Range</output_type>
-                <radiation_type>ultrasound</radiation_type>
-                <frame_name>sonar_link</frame_name>
-            </plugin>
-        </sensor>
-    </gazebo>
+    <xacro:macro name="insert_sonar" params="base_name parent_name x y z mass">
+        <joint name="${base_name}_joint" type="fixed">
+            <parent link="${parent_name}"/>
+            <child link="${base_name}"/>
+            <origin xyz="${x} ${y} ${z}" rpy="0 0 0"/>
+        </joint>
+        <link name="${base_name}">
+            <visual>
+                <origin xyz="-0.005 0 0" rpy="0 ${pi/2} 0"/>
+                <geometry>
+                    <cylinder radius="0.015" length="0.01" />
+                </geometry>
+                <material name="blue"/>
+            </visual>
+            <collision>
+                <origin xyz="-0.005 0 0" rpy="0 ${pi/2} 0"/>
+                <geometry>
+                    <cylinder radius="0.015" length="0.01" />
+                </geometry>
+            </collision>
+            <xacro:inertial_cylinder mass="${mass}" length="0.01" radius="0.01">
+                <origin xyz="-0.005 0 0" rpy="0 0 0"/>
+            </xacro:inertial_cylinder>
+        </link>
+        <gazebo reference="${base_name}">
+            <material>Gazebo/Blue</material>
+            <sensor name="${base_name}" type="ray">
+                <always_on>true</always_on>
+                <visualize>false</visualize>
+                <pose>0.0 0 0.0 0 0 0</pose>
+                <update_rate>5</update_rate>
+                <ray>
+                    <scan>
+                        <horizontal>
+                        <samples>20</samples>
+                        <resolution>1</resolution>
+                        <min_angle>${-scan_angle * deg2rad}</min_angle>
+                        <max_angle>${scan_angle * deg2rad}</max_angle>
+                        </horizontal>
+                        <vertical>
+                        <samples>20</samples>
+                        <resolution>1</resolution>
+                        <min_angle>${-scan_angle * deg2rad}</min_angle>
+                        <max_angle>${scan_angle * deg2rad}</max_angle>
+                        </vertical>
+                    </scan>
+                    <range>
+                        <min>0.01</min>
+                        <max>2</max>
+                        <resolution>0.02</resolution>
+                    </range>
+                </ray>
+                <plugin name="${base_name}_plugin" filename="libgazebo_ros_ray_sensor.so">
+                    <ros>
+                        <namespace>sonar</namespace>
+                        <remapping>~/out:=range</remapping>
+                    </ros>
+                    <output_type>sensor_msgs/Range</output_type>
+                    <radiation_type>ultrasound</radiation_type>
+                    <frame_name>${base_name}</frame_name>
+                </plugin>
+            </sensor>
+        </gazebo>
+    </xacro:macro>
 </robot>
