Commit message: feat:updated ros2 control settings

File: mobo_bot_description/urdf/controllers/ros2_control.xacro (robot description, xacro)
@@ -23,5 +23,5 @@
                 <remapping>~/out:=joint_states</remapping>
             </ros>
-            <update_rate>50</update_rate>
+            <update_rate>30</update_rate>
             <joint_name>left_wheel_joint</joint_name>
             <joint_name>right_wheel_joint</joint_name>

File: mobo_bot_description/urdf/controllers/transmission_macros.xacro (robot description, xacro)
@@ -1,5 +1,5 @@
 <?xml version="1.0"?>
 <robot xmlns:xacro="http://www.ros.org/wiki/xacro" >
-    <xacro:macro name="wheel_transmission" params="joint_name">
+    <xacro:macro name="insert_wheel_transmission" params="joint_name">
         <joint name="${joint_name}">
             <command_interface name="velocity">

File: mobo_bot_description/urdf/robot_core.xacro (robot description, xacro)
@@ -107,5 +107,5 @@
         x="${-chassis_length/4}" y="0" z="${chassis_height+lidar_z_offset}"
         mass="0.08" samples="360"
-        min_angle="${-pi/2}" max_angle="${pi/2}"
+        min_angle="${-pi*2}" max_angle="${pi*2}"
         min_range="0.1" max_range="10"
         visualize="false"/>
