Commit message: added new design and readme

File: mobo_bot_description/urdf/controllers/gazebo_control.xacro (robot description, xacro)
@@ -8,9 +8,9 @@
             <right_joint>right_wheel_joint</right_joint>
             <!-- kinematics -->
-            <wheel_separation>0.3</wheel_separation>
-            <wheel_diameter>0.065</wheel_diameter>
+            <wheel_separation>0.214</wheel_separation>
+            <wheel_diameter>0.068</wheel_diameter>
             <!-- limits -->
-            <max_wheel_torque>50</max_wheel_torque>
-            <max_wheel_acceleration>4.0</max_wheel_acceleration>
+            <max_wheel_torque>20</max_wheel_torque>
+            <max_wheel_acceleration>2.0</max_wheel_acceleration>
             <command_topic>cmd_vel</command_topic>
             <!-- output -->

File: mobo_bot_description/urdf/controllers/gazebo_hw_ros2_control.xacro (robot description, xacro)
@@ -2,5 +2,5 @@
 <robot name="mobo_bot" xmlns:xacro="http://www.ros.org/wiki/xacro">
     <xacro:include filename="transmission_macros.xacro"/>
-    <ros2_control name="mobo_bot_diff_drive_ros2_control" type="system">
+    <ros2_control name="mobo_bot_diff_drive_gazebo_hw_ros2_control" type="system">
         <hardware>
             <plugin>gazebo_ros2_control/GazeboSystem</plugin>
@@ -15,4 +15,7 @@
             <robot_param_node>robot_state_publisher</robot_param_node>
             <parameters>$(find mobo_bot_description)/config/diff_drive_controller.yaml</parameters>
+            <ros>
+                <remapping>/diff_drive_controller/cmd_vel_unstamped:=/cmd_vel</remapping>
+            </ros>
         </plugin>
     </gazebo>

File: mobo_bot_description/urdf/other_parts/drive_wheel_macro.xacro (robot description, xacro)
@@ -25,8 +25,8 @@
             <mu1>1.0</mu1>
             <mu2>1.0</mu2>
-            <!-- <kp>${kp}</kp> -->
-            <!-- <kd>${kd}</kd> -->
+            <!-- <kp>1000000</kp> -->
+            <!-- <kd>0.001</kd> -->
+            <!-- <minDepth>0.001</minDepth> -->
             <!-- <fdir1>${fdir}</fdir1> -->
-            <!-- <minDepth>0.005</minDepth> -->
             <material>Gazebo/FlatBlack</material>
         </gazebo>
@@ -51,6 +51,6 @@
             <origin xyz="0 0 0" rpy="0 0 0"/>
                 <geometry>
-                    <!-- <cylinder radius="${radius}" length="${thickness}"/> -->
-                    <sphere radius="${radius}"/>
+                    <cylinder radius="${radius}" length="${thickness}"/>
+                    <!-- <sphere radius="${radius}"/> -->
                 </geometry>
             </collision>
@@ -94,13 +94,4 @@
                 <xacro:material_red/>
             </visual>
-            <!-- <collision>
-                <origin xyz="0 0 0" rpy="0 0 0"/>
-                <geometry>
-                    <cylinder radius="${(radius*1.2)/2}" length="${thickness*2}"/>
-                </geometry>
-            </collision>
-            <xacro:inertial_cylinder mass="0.01" radius="${(radius*1.2)/2}" length="${thickness+0.005}">
-                <origin xyz="0 0 0" rpy="0 0 0"/>
-            </xacro:inertial_cylinder> -->
         </link>
         <gazebo reference="${base_name}_rim">

File: mobo_bot_description/urdf/robot_core.xacro (robot description, xacro)
@@ -3,19 +3,18 @@
     <xacro:include filename="other_parts/box_with_fillet_macro.xacro"/>
     <xacro:include filename="other_parts/drive_wheel_macro.xacro"/>
-    <xacro:include filename="other_parts/face_macro.xacro"/>
+    <xacro:include filename="sensors/sonar.xacro"/>
     <xacro:include filename="sensors/lidar.xacro"/>
-    <xacro:include filename="sensors/imu.xacro"/>
-    <xacro:include filename="sensors/cam.xacro"/>
-    <xacro:include filename="sensors/sonar.xacro"/>
-    <xacro:property name="chassis_height" value="0.125"/>
-    <xacro:property name="chassis_length" value="0.3"/>
-    <xacro:property name="wheel_seperation" value="0.3"/>
-    <xacro:property name="chassis_mass" value="4.0"/>
-    <xacro:property name="wheel_radius" value="0.0325"/>
+    <!-- <xacro:include filename="sensors/imu.xacro"/> -->
+    <!-- <xacro:include filename="sensors/cam.xacro"/> -->
+    <xacro:property name="chassis_length" value="0.25"/>
+    <xacro:property name="chassis_width" value="0.18"/>
+    <xacro:property name="chassis_height" value="0.09"/>
+    <xacro:property name="chassis_mass" value="3.0"/>
+    <xacro:property name="wheel_seperation" value="0.214"/>
+    <xacro:property name="wheel_radius" value="0.034"/>
     <xacro:property name="wheel_width" value="0.026"/>
     <xacro:property name="wheel_mass" value="0.08"/>
-    <xacro:property name="castor_wheel_radius" value="${wheel_radius/2}"/>
+    <xacro:property name="castor_wheel_radius" value="0.025"/>
     <xacro:property name="castor_wheel_mass" value="0.04"/>
-    <xacro:property name="chassis_width" value="${wheel_seperation-wheel_width-0.01}"/>
     <!-- BASE LINK -->
     <!-- <base joint/> -->
@@ -27,12 +26,12 @@
         <parent link="base_link"/>
         <child link="chassis"/>
-        <origin xyz="0 0 ${wheel_radius}"/>
+        <origin xyz="0 0 ${wheel_radius*2}"/>
     </joint>
     <link name="chassis">
-        <xacro:insert_box_with_fillet x="${-chassis_length/8}" y="0" z="${chassis_height/2}"
+        <xacro:insert_box_with_fillet x="${-chassis_length/6}" y="0" z="${chassis_height/2}"
             size_x="${chassis_length}" size_y="${chassis_width}" size_z="${chassis_height}"
-            fillet_radius="0.05" material="orange"/>
+            fillet_radius="0.04" material="orange"/>
         <collision>
-           <origin xyz="${-chassis_length/8} 0 ${chassis_height/2}" rpy="0 0 0"/>
+           <origin xyz="${-chassis_length/6} 0 ${chassis_height/2}" rpy="0 0 0"/>
             <geometry>
                 <box size="${chassis_length} ${chassis_width} ${chassis_height}"/>
@@ -40,5 +39,5 @@
         </collision>
         <xacro:inertial_box mass="${chassis_mass}" x="${chassis_length}" y="${chassis_width}" z="${chassis_height}">
-            <origin xyz="${-chassis_length/8} 0 ${chassis_height/2}" rpy="0 0 0"/>
+            <origin xyz="${-chassis_length/6} 0 ${wheel_radius*2}" rpy="0 0 0"/>
         </xacro:inertial_box>
     </link>
@@ -46,5 +45,5 @@
         <material>Gazebo/Orange</material>
     </gazebo>
-    <xacro:insert_face parent_name="chassis" x="${(chassis_length/8)*3}" y="0" z="${chassis_height/2}"/>
+    <!-- <xacro:insert_face parent_name="chassis" x="${(chassis_length/6)*2}" y="0" z="${chassis_height/2}"/> -->
     <!--  ########################### -->
     <!-- LEFT AND RIGHT DRIVE WHEELS -->
@@ -52,5 +51,5 @@
         base_name="left_wheel"
         parent_name="chassis"
-        x="0" y="${wheel_seperation/2}" z="0"
+        x="0" y="${wheel_seperation/2}" z="${-wheel_radius}"
         mass="${wheel_mass}"
         radius="${wheel_radius}"
@@ -60,5 +59,5 @@
         base_name="right_wheel"
         parent_name="chassis"
-        x="0" y="${-wheel_seperation/2}" z="0"
+        x="0" y="${-wheel_seperation/2}" z="${-wheel_radius}"
         mass="${wheel_mass}"
         radius="${wheel_radius}"
@@ -70,5 +69,5 @@
         <parent link="chassis"/>
         <child link="castor_wheel"/>
-        <origin xyz="${-chassis_length/2} 0 ${-wheel_radius/2}"/>
+        <origin xyz="${-chassis_length/2} 0 ${-1*((wheel_radius*2)-castor_wheel_radius)}"/>
     </joint>
     <link name="castor_wheel">
@@ -76,5 +75,5 @@
             <origin xyz="0 0 0" rpy="0 0 0"/>
             <geometry>
-                <sphere radius="${wheel_radius/2}" />
+                <sphere radius="${castor_wheel_radius}" />
             </geometry>
             <material name="silver"/>
@@ -83,8 +82,8 @@
            <origin xyz="0 0 0" rpy="0 0 0"/>
             <geometry>
-                <sphere radius="${wheel_radius/2}" />
+                <sphere radius="${castor_wheel_radius}" />
             </geometry>
         </collision>
-        <xacro:inertial_sphere mass="${castor_wheel_mass}" radius="${wheel_radius/2}">
+        <xacro:inertial_sphere mass="${castor_wheel_mass}" radius="${castor_wheel_radius}">
             <origin xyz="0 0 0" rpy="0 0 0"/>
         </xacro:inertial_sphere>
@@ -100,42 +99,32 @@
     </gazebo>
     <!--  ########################### -->
-    <!--  lidar -->
-    <xacro:property name="lidar_z_offset" value="0.1"/>
+    <!--  sonar -->
+    <xacro:insert_sonar
+        base_name="sonar"
+        parent_name="chassis"
+        x="${(chassis_length/6)*2}" y="0" z="${chassis_height/2}"
+        mass="0.0005"
+        min_range="0.02" max_range="3.0"
+        resolution="0.01" visualize="false"/>
+     <!--  lidar -->
+    <xacro:property name="lidar_z_offset" value="0.04"/>
     <xacro:insert_lidar
         base_name="lidar"
         parent_name="chassis"
-        x="${-chassis_length/4}" y="0" z="${chassis_height+lidar_z_offset}"
-        mass="0.08" samples="360"
+        x="${-chassis_length/3}" y="0" z="${chassis_height+lidar_z_offset}"
+        mass="0.1" samples="360"
         min_angle="${-pi*2}" max_angle="${pi*2}"
         min_range="0.1" max_range="10"
         visualize="false"/>
     <!--  imu -->
-    <xacro:insert_imu
+    <!-- <xacro:insert_imu
         base_name="imu"
         parent_name="chassis"
-        x="0" y="0" z="${chassis_height}"/>
-    <!--  line tracking camera style -->
-    <!-- <xacro:insert_camera
-        base_name="line_cam"
-        parent_name="chassis"
-        x="${(chassis_length*0.375)+0.03}" y="0" z="${0.05-wheel_radius}"
-        mass="0.005"
-        width="320" height="240"
-        min_range="0.02" max_range="5.0"
-        tilt_angle="${pi/2.1}"
-        visualize="false"/> -->
-    <!--  front sonar sensor -->
-    <!-- <xacro:insert_sonar
-        base_name="sonar"
-        parent_name="chassis"
-        x="${(chassis_length*0.375)+0.005}" y="0" z="${(chassis_height/2)+0.04}"
-        mass="0.0005"
-        min_range="0.02" max_range="3.0"
-        resolution="0.01" visualize="false"/> -->
-    <!--  normal camera style -->
+        x="0" y="0" z="${chassis_height}"/> -->
+    <!-- camera -->
     <!-- <xacro:property name="cam_x_offset" value="0.04"/>
     <xacro:property name="cam_z_offset" value="0.02"/>
     <xacro:insert_camera
-        base_name="line_cam"
+        base_name="camera"
         parent_name="chassis"
         x="${(chassis_length*0.375)+cam_x_offset}" y="0" z="${chassis_height+cam_z_offset}"
@@ -145,11 +134,3 @@
         tilt_angle="0"
         visualize="true"/> -->
-    <!--  front sonar sensor -->
-    <!-- <xacro:insert_sonar
-        base_name="sonar"
-        parent_name="chassis"
-        x="${(chassis_length*0.375)+0.005}" y="0" z="${(chassis_height/2)}"
-        mass="0.0005"
-        min_range="0.02" max_range="3.0"
-        resolution="0.01" visualize="false"/> -->
 </robot>

File: mobo_bot_description/urdf/robot_urdf.xacro (robot description, xacro)
@@ -3,9 +3,4 @@
     <!-- ########### ARGUMENTS ######################### -->
     <xacro:arg name="use_ros2_control" default="false"/>
-    <!-- <xacro:arg name="gazebo_visual" default="true"/> -->
-    <!-- <xacro:arg name="laser_visual" default="false"/> -->
-    <!-- <xacro:arg name="imu_visual"   default="true"/> -->
-    <!-- <xacro:arg name="sonar_visual"   default="false"/> -->
-    <!-- <xacro:arg name="cam_visual"   default="false"/> -->
     <!-- ############################################### -->
     <xacro:include filename="color_macros.xacro" />
@@ -13,12 +8,8 @@
     <xacro:include filename="robot_core.xacro" />
     <xacro:if value="$(arg use_ros2_control)">
-        <xacro:include filename="controllers/ros2_control.xacro" />
+        <xacro:include filename="controllers/gazebo_hw_ros2_control.xacro" />
     </xacro:if>
     <xacro:unless value="$(arg use_ros2_control)">
         <xacro:include filename="controllers/gazebo_control.xacro" />
     </xacro:unless>
-    <!-- <xacro:include filename="sensors/lidar.xacro" /> -->
-    <!-- <xacro:include filename="sensors/imu.xacro" /> -->
-    <!-- <xacro:include filename="sensors/camera.xacro" /> -->
-    <!-- <xacro:include filename="other_parts/face_macro.xacro" /> -->
 </robot>

File: mobo_bot_description/urdf/sensors/cam.xacro (robot description, xacro)
@@ -40,39 +40,69 @@
         <link name="${base_name}_optical_link"/>
         <gazebo reference="${base_name}">
-            <material>Gazebo/DarkGrey</material>
-            <sensor type="${base_name}" name="camera">
-                <visualize>${visualize}</visualize>
-                <update_rate>20.0</update_rate>
-                <camera name="${base_name}">
-                    <horizontal_fov>1.4</horizontal_fov>
-                    <image>
-                        <width>${width}</width>
-                        <height>${height}</height>
-                        <format>R8G8B8</format>
-                    </image>
-                    <clip>
-                        <near>${min_range}</near>
-                        <far>${max_range}</far>
-                    </clip>
-                    <noise>
-                        <type>gaussian</type>
-                        <mean>0.0</mean>
-                        <stddev>0.007</stddev>
-                    </noise>
-                </camera>
-                <plugin name="${base_name}_plugin" filename="libgazebo_ros_camera.so">
-                    <!-- <ros>
-                        <namespace>cam</namespace>
-                        <remapping>~/image_raw:=raw</remapping>
-                        <remapping>~/camera_info:=info</remapping>
-                    </ros> -->
-                    <!-- Set camera name. If empty, defaults to sensor name (i.e. "sensor_name") -->
-                    <camera_name>${base_name}</camera_name>
-                    <!-- Set TF frame name. If empty, defaults to link name (i.e. "link_name") -->
-                    <frame_name>${base_name}_optical_link</frame_name>
-                    <hack_baseline>0.2</hack_baseline>
-                </plugin>
-            </sensor>
+          <material>Gazebo/DarkGrey</material>
+          <sensor name="${base_name}" type="camera">
+            <pose> 0 0 0 0 0 0 </pose>
+            <visualize>${visualize}</visualize>
+            <update_rate>20</update_rate>
+            <camera>
+                <!-- <horizontal_fov>1.089</horizontal_fov> -->
+                <horizontal_fov>1.46608</horizontal_fov>
+                <image>
+                    <format>R8G8B8</format>
+                    <width>${width}</width>
+                    <height>${height}</height>
+                </image>
+                <clip>
+                    <near>${min_range}</near>
+                    <far>${max_range}</far>
+                </clip>
+            </camera>
+            <plugin name="${base_name}_plugin" filename="libgazebo_ros_camera.so">
+                <frame_name>${base_name}_optical_link</frame_name>
+            </plugin>
+          </sensor>
         </gazebo>
     </xacro:macro>
 </robot>
+ <!-- <joint name="line_cam_joint" type="fixed">
+        <parent link="chassis"/>
+        <child link="line_cam"/>
+        <origin xyz="0.305 0 0.08" rpy="0 0 0"/>
+    </joint>
+    <link name="line_cam">
+        <visual>
+            <geometry>
+                <box size="0.010 0.03 0.03"/>
+            </geometry>
+            <material name="red"/>
+        </visual>
+    </link>
+    <joint name="line_cam_optical_joint" type="fixed">
+        <parent link="line_cam"/>
+        <child link="line_cam_link_optical"/>
+        <origin xyz="0 0 0" rpy="${-pi/2} 0 ${-pi/2}"/>
+    </joint>
+    <link name="line_cam_link_optical"></link>
+    <gazebo reference="line_cam">
+        <material>Gazebo/Red</material>
+        <sensor name="line_cam" type="camera">
+            <pose> 0 0 0 0 0 0 </pose>
+            <visualize>true</visualize>
+            <update_rate>10</update_rate>
+            <camera>
+                <horizontal_fov>1.089</horizontal_fov>
+                <image>
+                    <format>R8G8B8</format>
+                    <width>640</width>
+                    <height>480</height>
+                </image>
+                <clip>
+                    <near>0.05</near>
+                    <far>8.0</far>
+                </clip>
+            </camera>
+            <plugin name="camera_controller" filename="libgazebo_ros_camera.so">
+                <frame_name>line_cam_link_optical</frame_name>
+            </plugin>
+        </sensor>
+    </gazebo> -->

File: mobo_bot_description/urdf/sensors/lidar.xacro (robot description, xacro)
@@ -9,24 +9,18 @@
         <link name="${base_name}">
             <visual>
-                <origin xyz="0 0 0"/>
+                <origin xyz="0 0 -0.02"/>
                 <geometry>
-                    <cylinder radius="0.05" length="0.04"/>
+                    <cylinder radius="0.03" length="0.04"/>
                 </geometry>
-                <material name="black"/>
-            </visual>
-            <visual>
-                <origin xyz="0 0 -0.05"/>
-                <geometry>
-                    <cylinder radius="0.01" length="0.1"/>
-                </geometry>
-                <material name="black"/>
+                <material name="grey"/>
             </visual>
             <collision>
+                <origin xyz="0 0 -0.02"/>
                 <geometry>
-                    <cylinder radius="0.05" length="0.04"/>
+                    <cylinder radius="0.03" length="0.04"/>
                 </geometry>
             </collision>
-            <xacro:inertial_cylinder mass="${mass}" length="0.04" radius="0.05">
-                <origin xyz="0 0 0" rpy="0 0 0"/>
+            <xacro:inertial_cylinder mass="${mass}" length="0.04" radius="0.03">
+                <origin xyz="0 0 -0.02" rpy="0 0 0"/>
             </xacro:inertial_cylinder>
         </link>

File: mobo_bot_description/urdf/sensors/sonar.xacro (robot description, xacro)
@@ -12,18 +12,31 @@
         <link name="${base_name}">
             <visual>
-                <origin xyz="-0.005 0 0" rpy="0 ${pi/2} 0"/>
+                <origin xyz="0 0.01 0" rpy="0 ${pi/2} 0"/>
                 <geometry>
-                    <cylinder radius="0.015" length="0.01" />
+                    <cylinder radius="0.006" length="0.006"/>
                 </geometry>
                 <material name="blue"/>
             </visual>
             <collision>
-                <origin xyz="-0.005 0 0" rpy="0 ${pi/2} 0"/>
+                <origin xyz="0 0.01 0" rpy="0 ${pi/2} 0"/>
                 <geometry>
-                    <cylinder radius="0.015" length="0.01" />
+                    <cylinder radius="0.006" length="0.006"/>
                 </geometry>
             </collision>
-            <xacro:inertial_cylinder mass="${mass}" length="0.01" radius="0.01">
-                <origin xyz="-0.005 0 0" rpy="0 0 0"/>
+            <visual>
+                <origin xyz="0 -0.01 0" rpy="0 ${pi/2} 0"/>
+                <geometry>
+                    <cylinder radius="0.006" length="0.006"/>
+                </geometry>
+                <material name="blue"/>
+            </visual>
+            <collision>
+                <origin xyz="0 -0.01 0" rpy="0 ${pi/2} 0"/>
+                <geometry>
+                    <cylinder radius="0.006" length="0.006"/>
+                </geometry>
+            </collision>
+            <xacro:inertial_cylinder mass="${mass}" length="0.006" radius="0.006">
+                <origin xyz="0 0.01 0" rpy="0 ${pi/2} 0"/>
             </xacro:inertial_cylinder>
         </link>
