Commit message: updated four standard wheel design

File: mobo_bot_description/urdf/controllers/gazebo_control.xacro (robot description, xacro)
@@ -2,28 +2,32 @@
 <robot xmlns:xacro="http://ros.org/wiki/xacro">
     <gazebo>
-        <plugin name="mobo_bot_diff_drive_gazebo_control" filename="libgazebo_ros_diff_drive.so">
-            <update_rate>40</update_rate>
+        <plugin name="mobo_bot_diff_skid_drive_gazebo_control" filename="libgazebo_ros_diff_drive.so">
             <!-- wheels -->
-            <left_joint>left_wheel_joint</left_joint>
-            <right_joint>right_wheel_joint</right_joint>
+            <num_wheel_pairs>2</num_wheel_pairs>
+            <left_joint>front_left_wheel_joint</left_joint>
+            <left_joint>rear_left_wheel_joint</left_joint>
+            <right_joint>front_right_wheel_joint</right_joint>
+            <right_joint>rear_right_wheel_joint</right_joint>
             <!-- kinematics -->
             <wheel_separation>0.214</wheel_separation>
+            <wheel_separation>0.214</wheel_separation>
+            <wheel_diameter>0.068</wheel_diameter>
             <wheel_diameter>0.068</wheel_diameter>
             <!-- limits -->
             <max_wheel_torque>20</max_wheel_torque>
             <max_wheel_acceleration>2.0</max_wheel_acceleration>
-            <command_topic>cmd_vel</command_topic>
-            <!-- output -->
+            <!-- odometry  -->
+            <!-- <odometry_source>world</odometry_source> -->
+            <odometry_frame>odom</odometry_frame>
+            <robot_base_frame>base_link</robot_base_frame>
+            <!-- topic & re remappings -->
+            <ros>
+              <!-- <namespace>/</namespace> -->
+              <!-- <remapping>/cmd_vel:=cmd_vel</remapping> -->
+              <!-- <remapping>/odom:=odom</remapping> -->
+            </ros>
             <publish_odom>true</publish_odom>
             <publish_odom_tf>true</publish_odom_tf>
-            <publish_wheel_tf>true</publish_wheel_tf>
-            <odometry_topic>odom</odometry_topic>
-            <odometry_frame>odom</odometry_frame>
-            <!-- <odometry_source>1</odometry_source> -->
-            <robot_base_frame>base_link</robot_base_frame>
-            <ros>
-                <!-- <namespace>/br</namespace> -->
-                <remapping>odom:=wheel/odometry</remapping>
-            </ros>
+            <update_rate>40.0</update_rate>
         </plugin>
     </gazebo>
@@ -34,7 +38,9 @@
                 <remapping>~/out:=joint_states</remapping>
             </ros>
-            <update_rate>30</update_rate>
-            <joint_name>left_wheel_joint</joint_name>
-            <joint_name>right_wheel_joint</joint_name>
+            <update_rate>50</update_rate>
+            <joint_name>front_left_wheel_joint</joint_name>
+            <joint_name>rear_left_wheel_joint</joint_name>
+            <joint_name>front_right_wheel_joint</joint_name>
+            <joint_name>rear_right_wheel_joint</joint_name>
         </plugin>
     </gazebo>

File: mobo_bot_description/urdf/controllers/gazebo_hw_ros2_control.xacro (robot description, xacro)
@@ -2,10 +2,17 @@
 <robot xmlns:xacro="http://www.ros.org/wiki/xacro">
     <xacro:include filename="transmission_macros.xacro"/>
-    <ros2_control name="mobo_bot_diff_drive_gazebo_hw_ros2_control" type="system">
+    <ros2_control name="mobo_bot_diff_drive_gazebo_hw_ros2_control_front" type="system">
         <hardware>
             <plugin>gazebo_ros2_control/GazeboSystem</plugin>
         </hardware>
-        <xacro:insert_wheel_transmission joint_name="left_wheel_joint"/>
-        <xacro:insert_wheel_transmission joint_name="right_wheel_joint"/>
+        <xacro:insert_wheel_transmission joint_name="front_left_wheel_joint"/>
+        <xacro:insert_wheel_transmission joint_name="front_right_wheel_joint"/>
+    </ros2_control>
+    <ros2_control name="mobo_bot_diff_drive_gazebo_hw_ros2_control_rear" type="system">
+        <hardware>
+            <plugin>gazebo_ros2_control/GazeboSystem</plugin>
+        </hardware>
+        <xacro:insert_wheel_transmission joint_name="rear_left_wheel_joint"/>
+        <xacro:insert_wheel_transmission joint_name="rear_right_wheel_joint"/>
     </ros2_control>
     <gazebo>
@@ -17,4 +24,5 @@
             <ros>
                 <remapping>/diff_drive_controller/cmd_vel_unstamped:=/cmd_vel</remapping>
+                <remapping>/diff_drive_controller/odom:=/odom</remapping>
             </ros>
         </plugin>
@@ -26,7 +34,9 @@
                 <remapping>~/out:=joint_states</remapping>
             </ros>
-            <update_rate>30</update_rate>
-            <joint_name>left_wheel_joint</joint_name>
-            <joint_name>right_wheel_joint</joint_name>
+            <update_rate>50</update_rate>
+            <joint_name>front_left_wheel_joint</joint_name>
+            <joint_name>front_right_wheel_joint</joint_name>
+            <joint_name>rear_left_wheel_joint</joint_name>
+            <joint_name>rear_right_wheel_joint</joint_name>
         </plugin>
     </gazebo>

File: mobo_bot_description/urdf/robot_core.xacro (robot description, xacro)
@@ -30,9 +30,9 @@
     </joint>
     <link name="chassis">
-        <xacro:insert_box_with_fillet x="${-chassis_length/6}" y="0" z="${chassis_height/2}"
+        <xacro:insert_box_with_fillet x="0" y="0" z="${chassis_height/2}"
             size_x="${chassis_length}" size_y="${chassis_width}" size_z="${chassis_height}"
-            fillet_radius="0.05" material="orange"/>
+            fillet_radius="0.06" material="orange"/>
         <collision>
-           <origin xyz="${-chassis_length/6} 0 ${chassis_height/2}" rpy="0 0 0"/>
+           <origin xyz="0 0 ${chassis_height/2}" rpy="0 0 0"/>
             <geometry>
                 <box size="${chassis_length} ${chassis_width} ${chassis_height}"/>
@@ -40,5 +40,5 @@
         </collision>
         <xacro:inertial_box mass="${chassis_mass}" x="${chassis_length}" y="${chassis_width}" z="${chassis_height}">
-            <origin xyz="${-chassis_length/6} 0 ${wheel_radius*2}" rpy="0 0 0"/>
+            <origin xyz="0 0 ${wheel_radius}" rpy="0 0 0"/>
         </xacro:inertial_box>
     </link>
@@ -47,15 +47,15 @@
     </gazebo>
     <!--  ########################### -->
-    <!-- LEFT DRIVE WHEEL -->
+    <!-- FRONT LEFT DRIVE WHEEL -->
     <xacro:insert_drive_wheel
-        base_name="left_wheel"
+        base_name="front_left_wheel"
         parent_name="base_link"
-        x="0" y="${wheel_seperation/2}" z="${wheel_radius}"
+        x="0.05" y="${wheel_seperation/2}" z="${wheel_radius}"
         mass="${wheel_mass}"
         radius="${wheel_radius}"
         thickness="${wheel_width}"/>
     <xacro:insert_drive_wheel_rim
-        base_name="left_rim"
-        parent_name="left_wheel"
+        base_name="front_left_rim"
+        parent_name="front_left_wheel"
         x="0" y="0" z="0.001"
         radius="${wheel_radius}"
@@ -63,15 +63,31 @@
         spoke_width="0.005"/>
     <!-- ############################# -->
-    <!-- RIGHT DRIVE WHEEL -->
+    <!-- REAR LEFT DRIVE WHEEL -->
     <xacro:insert_drive_wheel
-        base_name="right_wheel"
+        base_name="rear_left_wheel"
         parent_name="base_link"
-        x="0" y="${-wheel_seperation/2}" z="${wheel_radius}"
+        x="-0.05" y="${wheel_seperation/2}" z="${wheel_radius}"
         mass="${wheel_mass}"
         radius="${wheel_radius}"
         thickness="${wheel_width}"/>
     <xacro:insert_drive_wheel_rim
-        base_name="right_rim"
-        parent_name="right_wheel"
+        base_name="rear_left_rim"
+        parent_name="rear_left_wheel"
+        x="0" y="0" z="0.001"
+        radius="${wheel_radius}"
+        thickness="${wheel_width}"
+        spoke_width="0.005"/>
+    <!-- ############################# -->
+    <!-- FRONT RIGHT DRIVE WHEEL -->
+    <xacro:insert_drive_wheel
+        base_name="front_right_wheel"
+        parent_name="base_link"
+        x="0.05" y="${-wheel_seperation/2}" z="${wheel_radius}"
+        mass="${wheel_mass}"
+        radius="${wheel_radius}"
+        thickness="${wheel_width}"/>
+    <xacro:insert_drive_wheel_rim
+        base_name="front_right_rim"
+        parent_name="front_right_wheel"
         x="0" y="0" z="-0.001"
         radius="${wheel_radius}"
@@ -79,43 +95,25 @@
         spoke_width="0.005"/>
     <!-- ############################# -->
-    <!--  castor WHEEL LINK -->
-    <joint name="castor_wheel_joint" type="fixed">
-        <parent link="base_link"/>
-        <child link="castor_wheel"/>
-        <origin xyz="${-chassis_length/2} 0 ${castor_wheel_radius}"/>
-    </joint>
-    <link name="castor_wheel">
-        <visual>
-            <origin xyz="0 0 0" rpy="0 0 0"/>
-            <geometry>
-                <sphere radius="${castor_wheel_radius}" />
-            </geometry>
-            <material name="silver"/>
-        </visual>
-        <collision>
-           <origin xyz="0 0 0" rpy="0 0 0"/>
-            <geometry>
-                <sphere radius="${castor_wheel_radius}" />
-            </geometry>
-        </collision>
-        <xacro:inertial_sphere mass="${castor_wheel_mass}" radius="${castor_wheel_radius}">
-            <origin xyz="0 0 0" rpy="0 0 0"/>
-        </xacro:inertial_sphere>
-    </link>
-    <gazebo reference="castor_wheel">
-        <mu1>0.001</mu1>
-        <mu2>0.001</mu2>
-        <!-- <kp>1000000.0</kp> -->
-        <!-- <kd>1.0</kd> -->
-        <!-- <fdir1>1 0 0</fdir1> -->
-        <!-- <minDepth>0.01</minDepth> -->
-        <material>Gazebo/Silver</material>
-    </gazebo>
-    <!--  ########################### -->
+    <!-- REAR RIGHT DRIVE WHEEL -->
+    <xacro:insert_drive_wheel
+        base_name="rear_right_wheel"
+        parent_name="base_link"
+        x="-0.05" y="${-wheel_seperation/2}" z="${wheel_radius}"
+        mass="${wheel_mass}"
+        radius="${wheel_radius}"
+        thickness="${wheel_width}"/>
+    <xacro:insert_drive_wheel_rim
+        base_name="rear_right_rim"
+        parent_name="rear_right_wheel"
+        x="0" y="0" z="-0.001"
+        radius="${wheel_radius}"
+        thickness="${wheel_width}"
+        spoke_width="0.005"/>
+    <!-- ############################# -->
     <!--  sonar -->
     <xacro:insert_sonar
         base_name="sonar"
         parent_name="chassis"
-        x="${(chassis_length/6)*2}" y="0" z="${chassis_height/2}"
+        x="${chassis_length/2}" y="0" z="${chassis_height/2}"
         mass="0.005"
         min_range="0.02" max_range="3.0"
@@ -126,5 +124,5 @@
         base_name="lidar"
         parent_name="chassis"
-        x="${-chassis_length/3}" y="0" z="${chassis_height+lidar_z_offset}"
+        x="${-chassis_length/6}" y="0" z="${chassis_height+lidar_z_offset}"
         mass="0.1" samples="360"
         min_angle="${-pi*2}" max_angle="${pi*2}"

Commit message: update code

File: mobo_bot_description/urdf/controllers/gazebo_control.xacro (robot description, xacro)
@@ -10,6 +10,6 @@
             <right_joint>rear_right_wheel_joint</right_joint>
             <!-- kinematics -->
-            <wheel_separation>0.214</wheel_separation>
-            <wheel_separation>0.214</wheel_separation>
+            <wheel_separation>0.22</wheel_separation>
+            <wheel_separation>0.22</wheel_separation>
             <wheel_diameter>0.068</wheel_diameter>
             <wheel_diameter>0.068</wheel_diameter>

File: mobo_bot_description/urdf/controllers/gazebo_hw_ros2_control.xacro (robot description, xacro)
@@ -7,7 +7,9 @@
         </hardware>
         <xacro:insert_wheel_transmission joint_name="front_left_wheel_joint"/>
+        <xacro:insert_wheel_transmission joint_name="rear_left_wheel_joint"/>
         <xacro:insert_wheel_transmission joint_name="front_right_wheel_joint"/>
+        <xacro:insert_wheel_transmission joint_name="rear_right_wheel_joint"/>
     </ros2_control>
-    <ros2_control name="mobo_bot_diff_drive_gazebo_hw_ros2_control_rear" type="system">
+    <!-- <ros2_control name="mobo_bot_diff_drive_gazebo_hw_ros2_control_rear" type="system">
         <hardware>
             <plugin>gazebo_ros2_control/GazeboSystem</plugin>
@@ -15,5 +17,5 @@
         <xacro:insert_wheel_transmission joint_name="rear_left_wheel_joint"/>
         <xacro:insert_wheel_transmission joint_name="rear_right_wheel_joint"/>
-    </ros2_control>
+    </ros2_control> -->
     <gazebo>
         <plugin filename="libgazebo_ros2_control.so" name="gazebo_ros2_control">
@@ -36,6 +38,6 @@
             <update_rate>50</update_rate>
             <joint_name>front_left_wheel_joint</joint_name>
+            <joint_name>rear_left_wheel_joint</joint_name>
             <joint_name>front_right_wheel_joint</joint_name>
-            <joint_name>rear_left_wheel_joint</joint_name>
             <joint_name>rear_right_wheel_joint</joint_name>
         </plugin>

File: mobo_bot_description/urdf/robot_core.xacro (robot description, xacro)
@@ -12,5 +12,5 @@
     <xacro:property name="chassis_height" value="0.07"/>
     <xacro:property name="chassis_mass" value="3.0"/>
-    <xacro:property name="wheel_seperation" value="0.214"/>
+    <xacro:property name="wheel_seperation" value="0.22"/>
     <xacro:property name="wheel_radius" value="0.034"/>
     <xacro:property name="wheel_width" value="0.026"/>
@@ -27,5 +27,5 @@
         <parent link="base_link"/>
         <child link="chassis"/>
-        <origin xyz="0 0 ${(wheel_radius*2)+0.002}"/>
+        <origin xyz="0 0 ${wheel_radius}"/>
     </joint>
     <link name="chassis">
@@ -40,5 +40,5 @@
         </collision>
         <xacro:inertial_box mass="${chassis_mass}" x="${chassis_length}" y="${chassis_width}" z="${chassis_height}">
-            <origin xyz="0 0 ${wheel_radius}" rpy="0 0 0"/>
+            <origin xyz="0 0 ${wheel_radius/2}" rpy="0 0 0"/>
         </xacro:inertial_box>
     </link>
@@ -51,5 +51,5 @@
         base_name="front_left_wheel"
         parent_name="base_link"
-        x="0.05" y="${wheel_seperation/2}" z="${wheel_radius}"
+        x="0.04" y="${wheel_seperation/2}" z="${wheel_radius}"
         mass="${wheel_mass}"
         radius="${wheel_radius}"
@@ -67,5 +67,5 @@
         base_name="rear_left_wheel"
         parent_name="base_link"
-        x="-0.05" y="${wheel_seperation/2}" z="${wheel_radius}"
+        x="-0.04" y="${wheel_seperation/2}" z="${wheel_radius}"
         mass="${wheel_mass}"
         radius="${wheel_radius}"
@@ -83,5 +83,5 @@
         base_name="front_right_wheel"
         parent_name="base_link"
-        x="0.05" y="${-wheel_seperation/2}" z="${wheel_radius}"
+        x="0.04" y="${-wheel_seperation/2}" z="${wheel_radius}"
         mass="${wheel_mass}"
         radius="${wheel_radius}"
@@ -99,5 +99,5 @@
         base_name="rear_right_wheel"
         parent_name="base_link"
-        x="-0.05" y="${-wheel_seperation/2}" z="${wheel_radius}"
+        x="-0.04" y="${-wheel_seperation/2}" z="${wheel_radius}"
         mass="${wheel_mass}"
         radius="${wheel_radius}"
